Commit message: collision and inertia added in urdf

File: description/robot.urdf.xacro (robot description, xacro)
@@ -1,109 +1,4 @@
 <?xml version="1.0"?>
-<robot xmlns:xacro="http://www.ros.org/wiki/xacro"  name="robot">
-    <!-- Configurable Values -->
-    <!-- Base -->
-    <xacro:property name="base_length" value="0.1" />
-    <xacro:property name="base_radius" value="0.1" />
-    <!-- Link1 -->
-    <xacro:property name="shoulder_length" value="0.1" />
-    <xacro:property name="shoulder_radius" value="0.07" />
-    <!-- Link2 -->
-    <xacro:property name="upperarm_length" value="0.2" />
-    <xacro:property name="upperarm_radius" value="0.06" />
-    <!-- Link3 -->
-    <xacro:property name="elbow_length" value="0.05" />
-    <xacro:property name="elbow_radius" value="0.05" />
-    <!-- Link4 -->
-    <xacro:property name="forearm_length" value="0.1" />
-    <xacro:property name="forearm_radius" value="0.05" />
-    <!-- Gripper -->
-    <xacro:property name="gripper_length" value="0.05" />
-    <!-- LINKS AND JOINTS START HERE -->
-    <link name="world"></link>
-    <joint name="base_joint" type="fixed">
-        <parent link="world"/>
-        <child link="base"/>
-        <origin xyz="0 1 0" rpy="0 0 0"/>
-    </joint>
-    <link name="base">
-        <visual>
-            <origin xyz="0 0 ${base_length/2}" rpy="0 0 0"/>
-            <geometry>
-                <cylinder length="${base_length}" radius="${base_radius}"/>
-            </geometry>
-        </visual>
-    </link>
-    <joint name="shoulder_joint" type="revolute">
-        <parent link="base"/>
-        <child link="shoulder"/>
-        <origin xyz="0 0 ${base_length}" rpy="0 0 0"/>
-        <axis xyz="0 0 1"/>
-        <limit lower="-3.1416" upper="3.1416" effort="100" velocity="0.1"/>
-    </joint>
-    <link name="shoulder">
-        <visual>
-            <origin xyz="0 0 ${shoulder_length/2}" rpy="0 0 0"/>
-            <geometry>
-                <cylinder length="${shoulder_length}" radius="${shoulder_radius}"/>
-            </geometry>
-        </visual>
-    </link>
-    <joint name="upperarm_joint" type="revolute">
-        <parent link="shoulder"/>
-        <child link="upperarm"/>
-        <origin xyz="0 0 ${shoulder_length}" rpy="0 0 0"/>
-        <axis xyz="1 0 0"/>
-        <limit lower="-3.1416" upper="3.1416" effort="100" velocity="0.1"/>
-    </joint>
-    <link name="upperarm">
-        <visual>
-            <origin xyz="0 0 ${upperarm_length/2}" rpy="0 0 0"/>
-            <geometry>
-                <cylinder length="${upperarm_length}" radius="${upperarm_radius}"/>
-            </geometry>
-        </visual>
-    </link>
-    <joint name="elbow_joint" type="revolute">
-        <parent link="upperarm"/>
-        <child link="elbow"/>
-        <origin xyz="0 0 ${upperarm_length}" rpy="0 0 0"/>
-        <axis xyz="1 0 0"/>
-        <limit lower="-3.1416" upper="3.1416" effort="100" velocity="0.1"/>
-    </joint>
-    <link name="elbow">
-        <visual>
-            <origin xyz="0 0 ${elbow_length/2}" rpy="0 0 0"/>
-            <geometry>
-                <cylinder length="${elbow_length}" radius="${elbow_radius}"/>
-            </geometry>
-        </visual>
-    </link>
-    <joint name="forearm_joint" type="revolute">
-        <parent link="elbow"/>
-        <child link="forearm"/>
-        <origin xyz="0 0 ${elbow_length}" rpy="0 0 0"/>
-        <axis xyz="0 0 1"/>
-        <limit lower="-3.1416" upper="3.1416" effort="100" velocity="0.1"/>
-    </joint>
-    <link name="forearm">
-        <visual>
-            <origin xyz="0 0 ${forearm_length/2}" rpy="0 0 0"/>
-            <geometry>
-                <cylinder length="${forearm_length}" radius="${forearm_radius}"/>
-            </geometry>
-        </visual>
-    </link>
-    <joint name="gripper_joint" type="fixed">
-        <parent link="forearm"/>
-        <child link="gripper"/>
-        <origin xyz="0 0 ${forearm_length}" rpy="0 0 0"/>
-    </joint>
-    <link name="gripper">
-        <visual>
-            <origin xyz="0 0 ${gripper_length/2}" rpy="0 0 0"/>
-            <geometry>
-                <box size="${gripper_length} ${gripper_length} ${gripper_length}"/>
-            </geometry>
-        </visual>
-    </link>
+<robot xmlns:xacro="http://www.ros.org/wiki/xacro" name="robot">
+    <xacro:include filename="robot_arm.xacro" />
 </robot>

Commit message: tried setting up ros2_control

File: description/robot.urdf.xacro (robot description, xacro)
@@ -2,3 +2,4 @@
 <robot xmlns:xacro="http://www.ros.org/wiki/xacro" name="robot">
     <xacro:include filename="robot_arm.xacro" />
+    <xacro:include filename="ros2_control.xacro" />
 </robot>

File: description/robot_arm.xacro (robot description, xacro)
@@ -2,4 +2,23 @@
 <robot xmlns:xacro="http://www.ros.org/wiki/xacro">
     <xacro:include filename="inertial_macros.xacro" />
+    <!-- Materials for Color -->
+    <material name="white">
+        <color rgba="1 1 1 1"/>
+    </material>
+    <material name="red">
+        <color rgba="1 0 0 1"/>
+    </material>
+    <material name="yellow">
+        <color rgba="1 1 0 1"/>
+    </material>
+    <material name="sky_blue">
+        <color rgba="0.529 0.808 0.922 1"/>
+    </material>
+    <material name="green">
+        <color rgba="0 1 0 1"/>
+    </material>
+    <material name="purple">
+        <color rgba="0.902 0.902 0.980 1"/>
+    </material>
     <!-- Configurable Values -->
     <!-- Base -->
@@ -33,4 +52,5 @@
                 <cylinder length="${base_length}" radius="${base_radius}"/>
             </geometry>
+            <material name="white"/>
         </visual>
         <collision>
@@ -44,4 +64,8 @@
         </xacro:inertial_cylinder>
     </link>
+    <gazebo reference="base">
+        <material>Gazebo/White</material>
+    </gazebo>
+    <!-- =================================================================================== -->
     <joint name="shoulder_joint" type="revolute">
         <parent link="base"/>
@@ -57,4 +81,5 @@
                 <cylinder length="${shoulder_length}" radius="${shoulder_radius}"/>
             </geometry>
+            <material name="red"/>
         </visual>
         <collision>
@@ -68,4 +93,8 @@
         </xacro:inertial_cylinder>
     </link>
+    <gazebo reference="shoulder">
+        <material>Gazebo/Red</material>
+    </gazebo>
+    <!-- =================================================================================== -->
     <joint name="upperarm_joint" type="revolute">
         <parent link="shoulder"/>
@@ -81,4 +110,5 @@
                 <cylinder length="${upperarm_length}" radius="${upperarm_radius}"/>
             </geometry>
+            <material name="yellow"/>
         </visual>
         <collision>
@@ -92,4 +122,8 @@
         </xacro:inertial_cylinder>
     </link>
+    <gazebo reference="upperarm">
+        <material>Gazebo/Yellow</material>
+    </gazebo>
+    <!-- =================================================================================== -->
     <joint name="elbow_joint" type="revolute">
         <parent link="upperarm"/>
@@ -105,4 +139,5 @@
                 <cylinder length="${elbow_length}" radius="${elbow_radius}"/>
             </geometry>
+            <material name="sky_blue"/>
         </visual>
         <collision>
@@ -116,4 +151,8 @@
         </xacro:inertial_cylinder>
     </link>
+    <gazebo reference="elbow">
+        <material>Gazebo/SkyBlue</material>
+    </gazebo>
+    <!-- =================================================================================== -->
     <joint name="forearm_joint" type="revolute">
         <parent link="elbow"/>
@@ -129,4 +168,5 @@
                 <cylinder length="${forearm_length}" radius="${forearm_radius}"/>
             </geometry>
+            <material name="green"/>
         </visual>
         <collision>
@@ -140,4 +180,8 @@
         </xacro:inertial_cylinder>
     </link>
+    <gazebo reference="forearm">
+        <material>Gazebo/Green</material>
+    </gazebo>
+    <!-- =================================================================================== -->
     <joint name="gripper_joint" type="fixed">
         <parent link="forearm"/>
@@ -151,4 +195,5 @@
                 <box size="${gripper_length} ${gripper_length} ${gripper_length}"/>
             </geometry>
+            <material name="purple"/>
         </visual>
         <collision>
@@ -162,3 +207,7 @@
         </xacro:inertial_box>
     </link>
+    <gazebo reference="gripper">
+        <material>Gazebo/Purple</material>
+    </gazebo>
+    <!-- =================================================================================== -->
 </robot>
